File: docs/static/circuito-elétrico/circuito-elétrico.kicad_sch (KiCad schematic)
At the start: 4 parts, among them J1 Conn_01x01_Pin, J2 Conn_01x01_Pin, J3 Conn_01x01_Pin, J4 Conn_01x01_Pin

Commit message: diagrama final
Parts:
- removed J3, J4: Conn_01x01_Pin, symbol Connector:Conn_01x01_Pin
- added U1: RP2040, Package_DFN_QFN:QFN-56-1EP_7x7mm_P0.4mm_EP3.2x3.2mm, symbol MCU_RaspberryPi:RP2040
Connections:
- net GP2: now reaches J2.1 (Pin_1)
- net GP2: now also U1.4 (GPIO2)
- net GP3: now reaches J1.1 (Pin_1)
- net GP3: now also U1.5 (GPIO3)
- new net: U1.1 (IOVDD), U1.10 (IOVDD), U1.22 (IOVDD), U1.33 (IOVDD), U1.42 (IOVDD), U1.49 (IOVDD)
- new net: U1.23 (DVDD), U1.50 (DVDD)
Other:
- note added: "Cabo da câmera"
- note added: "Câmera USB"
- note removed: "GP2"
- note removed: "GP3"
- moved on the sheet: J1, J2
